File: kicad/hcms_dot_display/_autosave-hcms_dot_display.kicad_sch (KiCad schematic)
At the start: 42 parts, among them J1 Conn_01x11, J2 USB_C_Receptacle_USB2.0, J3 Conn_01x11, J4 Conn_01x10_Female, J5 Conn_01x10_Male, J6 Conn_01x10_Male, J7 Conn_01x10_Female, Q1 Q_PMOS_DSG, Q2 Q_PMOS_DSG, Q3 Q_PMOS_DSG, Q4 Q_PMOS_DSG, Q5 Q_PMOS_DSG, SW2 SW_SPST, U1 ATtiny826-SXX, U2 FT231XS

Commit message: pughe
Parts:
- added SW?: SW_DIP_x03, symbol Switch:SW_DIP_x03
Changed lines of the file:
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@@
     (pin "2")
+  )
+  (symbol (lib_id "Switch:SW_DIP_x03") (at 118.11 173.99 0) (unit 1)
+    (in_bom yes) (on_board yes) (fields_autoplaced)
+    (property "Reference" "SW?" (id 0) (at 118.11 161.29 0))
+    (property "Value" "SW_DIP_x03" (id 1) (at 118.11 163.83 0))
+    (property "Footprint" "" (id 2) (at 118.11 173.99 0)
+      (effects (font (size 1.27 1.27)) hide)
+    )
+    (property "Datasheet" "~" (id 3) (at 118.11 173.99 0)
+      (effects (font (size 1.27 1.27)) hide)
+    )
+    (pin "1")
+    (pin "2")
+    (pin "3")
+    (pin "4")
+    (pin "5")
+    (pin "6")
   )
   (symbol (lib_id "Device:R") (at 158.75 198.12 270) (unit 1)
@@
       (reference "SW2") (unit 1) (value "SW_SPST") (footprint "Button_Switch_SMD:SW_DIP_SPSTx03_Slide_KingTek_DSHP03TS_W7.62mm_P1.27mm")
     )
+    (path "/ae986f85-a96b-434a-bd76-aa65361451aa"
+      (reference "SW?") (unit 1) (value "SW_DIP_x03") (footprint "")
+    )
     (path "/ec702393-b640-4b47-ba2e-5eeb75d59724"
