File: kicad/hcms_dot_display/hcms_dot_display.kicad_sch (KiCad schematic)
At the start: 42 parts, among them J1 Conn_01x11, J2 USB_C_Receptacle_USB2.0, J3 Conn_01x11, J4 Conn_01x10_Female, J5 Conn_01x10_Male, J6 Conn_01x10_Male, J7 Conn_01x10_Female, Q1 Q_PMOS_DSG, Q2 Q_PMOS_DSG, Q3 Q_PMOS_DSG, Q4 Q_PMOS_DSG, Q5 Q_PMOS_DSG, SW2 SW_SPST, U1 ATtiny826-SXX, U2 FT231XS

Commit message: Added Vcol rail and switching PMOS.  Started new board to board cons
Parts:
- removed J1: Conn_01x11, hcms:input board to board con, symbol Connector_Generic:Conn_01x11
- removed J3: Conn_01x11, hcms:output board to board con, symbol Connector_Generic:Conn_01x11
- added C12: 100nF, Capacitor_SMD:C_0603_1608Metric, symbol Device:C_Small
- added J1: (no value), symbol Connector_Generic:Conn_01x12
- added J3: Conn_01x12, hcms:input board to board con top bot, symbol Connector_Generic:Conn_01x12
- added Q6: (no value), symbol Device:Q_PMOS_DSG
- added R3: 200, Resistor_SMD:R_0603_1608Metric, symbol Device:R
Connections:
- net +5V: now also J1.1 (Pin_1), J3.1 (Pin_1), Q6.2 (S); no longer Q1.2 (S), Q2.2 (S), Q3.2 (S), Q4.2 (S), Q5.2 (S)
- net CLK: now also J1.9 (Pin_9), J3.9 (Pin_9)
- net COL_PWM: now also R3.1
- net DAISY_A_DATA: now also J1.10 (Pin_10), J3.10 (Pin_10)
- net DAISY_B_DATA: now also J1.11 (Pin_11), J3.11 (Pin_11)
- net GND: now also C12.2, J1.12 (Pin_12), J3.12 (Pin_12)
- net MCU_COL_1: now also J1.3 (Pin_3), J3.3 (Pin_3)
- net MCU_COL_2: now also J1.4 (Pin_4), J3.4 (Pin_4)
- net MCU_COL_3: now also J1.5 (Pin_5), J3.5 (Pin_5)
- net MCU_COL_4: now also J1.6 (Pin_6), J3.6 (Pin_6)
- net MCU_COL_5: now also J1.7 (Pin_7), J3.7 (Pin_7)
- net nBLNK: now also J1.8 (Pin_8), J3.8 (Pin_8)
- new net: Q6.3 (G), R3.2
- new net V_COL: C12.1, J1.2 (Pin_2), J3.2 (Pin_2), Q1.2 (S), Q2.2 (S), Q3.2 (S), Q4.2 (S), Q5.2 (S), Q6.1 (D)
Other:
- note added: "SI4425FDY-T1-GE3"
- moved on the sheet: Q1, Q2, Q3, Q4, Q5, R10, R11, R12, R13, R14

Commit message: literally in the middle of fixing left right conn but time to climb
Parts:
- removed J6: Conn_01x10_Male, Connector_PinHeader_2.54mm:PinHeader_1x10_P2.54mm_Vertical, symbol Connector:Conn_01x10_Male
- removed J7: Conn_01x10_Female, Connector_PinHeader_2.54mm:PinHeader_1x10_P2.54mm_Vertical, symbol Connector:Conn_01x10_Female
- added J6, J7: Conn_01x12, hcms:input board to board con top bot, symbol Connector_Generic:Conn_01x12
- J1: value (none) -> Conn_01x12; footprint (none) -> hcms:board to board con top bot
- J4: value Conn_01x10_Female -> Conn_01x11_Female; symbol Connector:Conn_01x10_Female -> Connector:Conn_01x11_Female
- J5: value Conn_01x10_Male -> Conn_01x11_Male; symbol Connector:Conn_01x10_Male -> Connector:Conn_01x11_Male
- Q6: value (none) -> Q_PMOS_DSG; footprint (none) -> Package_SO:SO-8_5.3x6.2mm_P1.27mm
Connections:
- net +5V: now also J6.1 (Pin_1), J7.1 (Pin_1)
- net CLK: now also J4.9 (Pin_9), J5.9 (Pin_9), J6.9 (Pin_9), J7.9 (Pin_9); no longer J4.8 (Pin_8), J5.8 (Pin_8)
- net DAISY_A_DATA: now also J6.10 (Pin_10), J7.10 (Pin_10)
- net DAISY_B_DATA: now also J6.11 (Pin_11), J7.11 (Pin_11)
- net GND: now also J4.11 (Pin_11), J5.11 (Pin_11), J6.12 (Pin_12), J7.12 (Pin_12); no longer J4.10 (Pin_10), J5.10 (Pin_10)
- net MCU_COL_1: now also J4.3 (Pin_3), J5.3 (Pin_3), J6.3 (Pin_3), J7.3 (Pin_3); no longer J4.2 (Pin_2), J5.2 (Pin_2)
- net MCU_COL_2: now also J4.4 (Pin_4), J5.4 (Pin_4), J6.4 (Pin_4), J7.4 (Pin_4); no longer J4.3 (Pin_3), J5.3 (Pin_3)
- net MCU_COL_3: now also J4.5 (Pin_5), J5.5 (Pin_5), J6.5 (Pin_5), J7.5 (Pin_5); no longer J4.4 (Pin_4), J5.4 (Pin_4)
- net MCU_COL_4: now also J4.6 (Pin_6), J5.6 (Pin_6), J6.6 (Pin_6), J7.6 (Pin_6); no longer J4.5 (Pin_5), J5.5 (Pin_5)
- net MCU_COL_5: now also J4.7 (Pin_7), J5.7 (Pin_7), J6.7 (Pin_7), J7.7 (Pin_7); no longer J4.6 (Pin_6), J5.6 (Pin_6)
- net MCU_DATA: now also J4.10 (Pin_10), J5.10 (Pin_10); no longer J4.9 (Pin_9), J5.9 (Pin_9)
- net V_COL: now also J4.2 (Pin_2), J5.2 (Pin_2), J6.2 (Pin_2), J7.2 (Pin_2)
- net nBLNK: now also J4.8 (Pin_8), J5.8 (Pin_8), J6.8 (Pin_8), J7.8 (Pin_8); no longer J4.7 (Pin_7), J5.7 (Pin_7)
Other:
- moved on the sheet: J1, J3

Commit message: beginning of ecos
Parts:
- added R16, R17: DNP, Resistor_SMD:R_0603_1608Metric, symbol Device:R
- J3: footprint hcms:input board to board con top bot -> hcms:board to board con top bot
- J4: footprint Connector_PinHeader_2.54mm:PinHeader_1x10_P2.54mm_Vertical -> Connector_PinSocket_2.54mm:PinSocket_1x11_P2.54mm_Vertical
- J5: footprint Connector_PinHeader_2.54mm:PinHeader_1x10_P2.54mm_Vertical -> Connector_PinHeader_2.54mm:PinHeader_1x11_P2.54mm_Vertical
- J6, J7: footprint hcms:input board to board con top bot -> hcms:board to board con left right
Connections:
- net A_DATA: now also J3.10 (Pin_10), J7.10 (Pin_10)
- net B_DATA: now also J3.11 (Pin_11), J7.11 (Pin_11)
- net DAISY_A_DATA: now also R17.2; no longer J3.10 (Pin_10), J7.10 (Pin_10)
- net DAISY_B_DATA: now also R16.2; no longer J3.11 (Pin_11), J7.11 (Pin_11)
- net at D1.26A (DATA_IN), R1.1, R2.1: now also R16.1
- net at D1.26B (DATA_IN), R6.1, R7.1: now also R17.1
Changed lines of the file:
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@@
   (junction (at 265.43 187.96) (diameter 0) (color 0 0 0 0)
   )
+  (junction (at 231.14 116.84) (diameter 0) (color 0 0 0 0)
+  )
   (junction (at 260.35 222.25) (diameter 0) (color 0 0 0 0)
   )
@@
   )
   (junction (at 141.605 40.005) (diameter 0) (color 0 0 0 0)
+  )
+  (junction (at 230.505 62.23) (diameter 0) (color 0 0 0 0)
   )
   (junction (at 136.525 208.915) (diameter 0) (color 0 0 0 0)
@@
     (stroke (width 0) (type default) (color 0 0 0 0))
   )
+  (wire (pts (xy 227.965 69.85) (xy 230.505 69.85))
+    (stroke (width 0) (type default) (color 0 0 0 0))
+  )
   (wire (pts (xy 374.65 121.92) (xy 374.65 118.11))
     (stroke (width 0) (type default) (color 0 0 0 0))
@@
     (stroke (width 0) (type default) (color 0 0 0 0))
   )
+  (wire (pts (xy 228.6 124.46) (xy 231.14 124.46))
+    (stroke (width 0) (type default) (color 0 0 0 0))
+  )
   (wire (pts (xy 379.73 121.92) (xy 379.73 118.11))
     (stroke (width 0) (type default) (color 0 0 0 0))
@@
     (stroke (width 0) (type default) (color 0 0 0 0))
   )
+  (wire (pts (xy 206.375 69.85) (xy 220.345 69.85))
+    (stroke (width 0) (type default) (color 0 0 0 0))
+  )
   (wire (pts (xy 369.57 121.92) (xy 369.57 118.11))
     (stroke (width 0) (type default) (color 0 0 0 0))
@@
     (stroke (width 0) (type default) (color 0 0 0 0))
   )
+  (wire (pts (xy 231.14 124.46) (xy 231.14 116.84))
+    (stroke (width 0) (type default) (color 0 0 0 0))
+  )
   (wire (pts (xy 120.015 59.69) (xy 133.985 59.69))
     (stroke (width 0) (type default) (color 0 0 0 0))
@@
     (stroke (width 0) (type default) (color 0 0 0 0))
   )
+  (wire (pts (xy 230.505 62.23) (xy 230.505 69.85))
+    (stroke (width 0) (type default) (color 0 0 0 0))
+  )
   (wire (pts (xy 286.385 80.645) (xy 299.085 80.645))
     (stroke (width 0) (type default) (color 0 0 0 0))
@@
   )
   (wire (pts (xy 372.11 121.92) (xy 372.11 118.11))
+    (stroke (width 0) (type default) (color 0 0 0 0))
+  )
+  (wire (pts (xy 207.01 124.46) (xy 220.98 124.46))
     (stroke (width 0) (type default) (color 0 0 0 0))
   )
@@
     (effects (font (size 1.27 1.27)) (justify left bottom))
   )
+  (label "DAISY_A_DATA" (at 207.01 124.46 0)
+    (effects (font (size 1.27 1.27)) (justify left bottom))
+  )
   (label "MCU_COL_3" (at 367.03 118.11 90)
     (effects (font (size 1.27 1.27)) (justify left bottom))
@@
     (effects (font (size 1.27 1.27)) (justify left bottom))
   )
-  (label "DAISY_A_DATA" (at 400.685 59.055 180)
+  (label "A_DATA" (at 400.685 59.055 180)
     (effects (font (size 1.27 1.27)) (justify right bottom))
   )
@@
     (effects (font (size 1.27 1.27)) (justify left bottom))
   )
-  (label "DAISY_A_DATA" (at 362.585 59.055 180)
+  (label "A_DATA" (at 362.585 59.055 180)
     (effects (font (size 1.27 1.27)) (justify right bottom))
   )
@@
     (effects (font (size 1.27 1.27)) (justify left bottom))
   )
-  (label "DAISY_B_DATA" (at 400.685 61.595 180)
+  (label "B_DATA" (at 400.685 61.595 180)
     (effects (font (size 1.27 1.27)) (justify right bottom))
   )
@@
     (effects (font (size 1.27 1.27)) (justify left bottom))
   )
+  (label "DAISY_B_DATA" (at 206.375 69.85 0)
+    (effects (font (size 1.27 1.27)) (justify left bottom))
+  )
   (label "MCU_COL_5" (at 340.36 219.71 180)
     (effects (font (size 1.27 1.27)) (justify right bottom))
@@
     (effects (font (size 1.27 1.27)) (justify left bottom))
   )
-  (label "DAISY_B_DATA" (at 362.585 61.595 180)
+  (label "B_DATA" (at 362.585 61.595 180)
     (effects (font (size 1.27 1.27)) (justify right bottom))
   )
@@
     (property "Reference" "J5" (id 0) (at 386.715 123.825 90))
     (property "Value" "Conn_01x11_Male" (id 1) (at 393.7 126.365 90))
-    (property "Footprint" "Connector_PinHeader_2.54mm:PinHeader_1x10_P2.54mm_Vertical" (id 2) (at 369.57 127 0)
+    (property "Footprint" "Connector_PinHeader_2.54mm:PinHeader_1x11_P2.54mm_Vertical" (id 2) (at 369.57 127 0)
       (effects (font (size 1.27 1.27)) hide)
     )
@@
   )
   (symbol (lib_id "Connector_Generic:Conn_01x12") (at 47.625 54.61 0) (unit 1)
-    (in_bom yes) (on_board yes) (fields_autoplaced)
+    (in_bom yes) (on_board yes)
     (property "Reference" "J1" (id 0) (at 50.8 54.6099 0)
       (effects (font (size 1.27 1.27)) (justify left))
@@
       (effects (font (size 1.27 1.27)) (justify left))
     )
-    (property "Footprint" "hcms:board to board con top bot" (id 2) (at 47.625 54.61 0)
-      (effects (font (size 1.27 1.27)) hide)
-    )
+    (property "Footprint" "hcms:board to board con top bot" (id 2) (at 67.31 59.69 0))
     (property "Datasheet" "~" (id 3) (at 47.625 54.61 0)
       (effects (font (size 1.27 1.27)) hide)
@@
     )
     (pin "1")
+  )
+  (symbol (lib_id "Device:R") (at 224.155 69.85 270) (unit 1)
+    (in_bom yes) (on_board yes)
+    (property "Reference" "R16" (id 0) (at 221.615 68.58 90)
+      (effects (font (size 1.27 1.27)) (justify left bottom))
+    )
+    (property "Value" "DNP" (id 1) (at 221.615 71.12 90)
+      (effects (font (size 1.27 1.27)) (justify left top))
+    )
+    (property "Footprint" "Resistor_SMD:R_0603_1608Metric" (id 2) (at 224.155 68.072 90)
+      (effects (font (size 1.27 1.27)) hide)
+    )
+    (property "Datasheet" "~" (id 3) (at 224.155 69.85 0)
+      (effects (font (size 1.27 1.27)) hide)
+    )
+    (pin "1")
+    (pin "2")
   )
   (symbol (lib_id "Device:C_Small") (at 147.32 205.105 0) (unit 1)
@@
       (effects (font (size 1.27 1.27)) (justify left))
     )
-    (property "Footprint" "Connector_PinHeader_2.54mm:PinHeader_1x10_P2.54mm_Vertical" (id 2) (at 369.57 140.97 0)
+    (property "Footprint" "Connector_PinSocket_2.54mm:PinSocket_1x11_P2.54mm_Vertical" (id 2) (at 369.57 140.97 0)
       (effects (font (size 1.27 1.27)) hide)
     )
@@
       (effects (font (size 1.27 1.27)) (justify left))
     )
-    (property "Footprint" "hcms:input board to board con top bot" (id 2) (at 338.455 48.895 0)
-      (effects (font (size 1.27 1.27)) hide)
-    )
+    (property "Footprint" "hcms:board to board con top bot" (id 2) (at 335.28 52.07 90))
     (property "Datasheet" "~" (id 3) (at 338.455 48.895 0)
       (effects (font (size 1.27 1.27)) hide)
@@
       (effects (font (size 1.27 1.27)) (justify left))
     )
-    (property "Footprint" "hcms:input board to board con top bot" (id 2) (at 376.555 48.895 0)
-      (effects (font (size 1.27 1.27)) hide)
-    )
+    (property "Footprint" "hcms:board to board con left right" (id 2) (at 373.38 52.705 90))
     (property "Datasheet" "~" (id 3) (at 376.555 48.895 0)
       (effects (font (size 1.27 1.27)) hide)
@@
   )
   (symbol (lib_id "Connector_Generic:Conn_01x12") (at 47.625 100.33 0) (unit 1)
-    (in_bom yes) (on_board yes) (fields_autoplaced)
+    (in_bom yes) (on_board yes)
     (property "Reference" "J6" (id 0) (at 50.8 100.3299 0)
       (effects (font (size 1.27 1.27)) (justify left))
@@
       (effects (font (size 1.27 1.27)) (justify left))
     )
-    (property "Footprint" "hcms:input board to board con top bot" (id 2) (at 47.625 100.33 0)
-      (effects (font (size 1.27 1.27)) hide)
-    )
+    (property "Footprint" "hcms:board to board con left right" (id 2) (at 67.945 105.41 0))
     (property "Datasheet" "~" (id 3) (at 47.625 100.33 0)
       (effects (font (size 1.27 1.27)) hide)
@@
     )
     (pin "1")
+  )
+  (symbol (lib_id "Device:R") (at 224.79 124.46 270) (unit 1)
+    (in_bom yes) (on_board yes)
+    (property "Reference" "R17" (id 0) (at 222.25 123.19 90)
+      (effects (font (size 1.27 1.27)) (justify left bottom))
+    )
+    (property "Value" "DNP" (id 1) (at 222.25 125.73 90)
+      (effects (font (size 1.27 1.27)) (justify left top))
+    )
+    (property "Footprint" "Resistor_SMD:R_0603_1608Metric" (id 2) (at 224.79 122.682 90)
+      (effects (font (size 1.27 1.27)) hide)
+    )
+    (property "Datasheet" "~" (id 3) (at 224.79 124.46 0)
+      (effects (font (size 1.27 1.27)) hide)
+    )
+    (pin "1")
+    (pin "2")
   )
   (symbol (lib_id "hcms_dot_display:ATtiny826-SXX") (at 307.34 205.74 0) (unit 1)
@@
     )
     (path "/cf0710a0-2c14-4971-a718-9e1eaa65f715"
-      (reference "J3") (unit 1) (value "Conn_01x12") (footprint "hcms:input board to board con top bot")
+      (reference "J3") (unit 1) (value "Conn_01x12") (footprint "hcms:board to board con top bot")
     )
     (path "/cab9e460-5933-40bb-ae00-cb8f811c254d"
-      (reference "J4") (unit 1) (value "Conn_01x11_Female") (footprint "Connector_PinHeader_2.54mm:PinHeader_1x10_P2.54mm_Vertical")
+      (reference "J4") (unit 1) (value "Conn_01x11_Female") (footprint "Connector_PinSocket_2.54mm:PinSocket_1x11_P2.54mm_Vertical")
     )
     (path "/4a10c4dc-bdfb-4468-97a7-ac6c0d3eeb26"
-      (reference "J5") (unit 1) (value "Conn_01x11_Male") (footprint "Connector_PinHeader_2.54mm:PinHeader_1x10_P2.54mm_Vertical")
+      (reference "J5") (unit 1) (value "Conn_01x11_Male") (footprint "Connector_PinHeader_2.54mm:PinHeader_1x11_P2.54mm_Vertical")
     )
     (path "/d575a104-8fac-4c40-b154-f41c50fe8c71"
-      (reference "J6") (unit 1) (value "Conn_01x12") (footprint "hcms:input board to board con top bot")
+      (reference "J6") (unit 1) (value "Conn_01x12") (footprint "hcms:board to board con left right")
     )
     (path "/d17dd236-9e69-4332-9741-17b1d82d4ff0"
-      (reference "J7") (unit 1) (value "Conn_01x12") (footprint "hcms:input board to board con top bot")
+      (reference "J7") (unit 1) (value "Conn_01x12") (footprint "hcms:board to board con left right")
     )
     (path "/cb19c6f6-ba2e-40c5-b24e-87d5c3df300e"
@@
       (reference "R15") (unit 1) (value "1k") (footprint "Resistor_SMD:R_0603_1608Metric")
     )
+    (path "/bb4b8dc1-a975-4a32-b8a6-91ad217d5079"
+      (reference "R16") (unit 1) (value "DNP") (footprint "Resistor_SMD:R_0603_1608Metric")
+    )
+    (path "/e7b4a87f-0a26-41f5-8b11-06bd54ddffc8"
+      (reference "R17") (unit 1) (value "DNP") (footprint "Resistor_SMD:R_0603_1608Metric")
+    )
     (path "/26df86c2-e6da-4304-8085-b1a7b60b8ac0"

Commit message: aidan im pushing
Parts:
- removed SW2: SW_SPST, Button_Switch_SMD:SW_DIP_SPSTx03_Slide_KingTek_DSHP03TS_W7.62mm_P1.27mm, symbol Switch:SW_SPST
- added R18, R19, R20: 10k, Resistor_SMD:R_0603_1608Metric, symbol Device:R
- added R21, R22: 0, Resistor_SMD:R_0603_1608Metric, symbol Device:R
- added SW1: SW_DIP_x03, symbol Switch:SW_DIP_x03
- R4, R5: value 10k -> 5.1k
Connections:
- net +5V: now also R21.1, SW1.1, SW1.2, SW1.3
- net GND: now also R18.1, R19.1, R20.1
- net V_COL: now also R22.1; no longer C12.1, Q6.1 (D)
- net at J2.A4 (VBUS), J2.A9 (VBUS), J2.B4 (VBUS)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: now also R21.2
- net CONFIG_0: now reaches U1.17 (PA1)
- net CONFIG_0: now also R18.2, SW1.6
- net CONFIG_1: now reaches U1.2 (PA4)
- net CONFIG_1: now also R19.2, SW1.5
- net CONFIG_2: now reaches U1.4 (PA6)
- net CONFIG_2: now also R20.2, SW1.4
- new net: C12.1, Q6.1 (D), R22.2
- no-connect marks 32 -> 36
Other:
- moved on the sheet: C1, C12, C2, J3, J4, J5, J7, Q6, R3, RV1, U1

Commit message: added switch fp, cleaned up placement. ready for routing
Parts:
- SW1: footprint (none) -> hcms:BPA03SB
Changed lines of the file:
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@@
     (property "Reference" "SW1" (id 0) (at 288.925 165.735 0))
     (property "Value" "SW_DIP_x03" (id 1) (at 288.925 168.275 0))
-    (property "Footprint" "" (id 2) (at 288.925 178.435 0)
+    (property "Footprint" "hcms:BPA03SB" (id 2) (at 288.925 178.435 0)
       (effects (font (size 1.27 1.27)) hide)
     )
@@
     )
     (path "/d65faba5-fee5-4bc2-bec5-3b7099da5631"
-      (reference "SW1") (unit 1) (value "SW_DIP_x03") (footprint "")
+      (reference "SW1") (unit 1) (value "SW_DIP_x03") (footprint "hcms:BPA03SB")
     )
     (path "/ec702393-b640-4b47-ba2e-5eeb75d59724"

Commit message: finally gonna start routing ??
Parts:
- Q6: symbol Device:Q_PMOS_DSG -> hcms_dot_display:SI4425FDY
Connections:
- net +5V: now also Q6.1 (S), Q6.3 (S)
- net MCU_COL_1: now also J4.5 (Pin_5), J5.5 (Pin_5); no longer J4.3 (Pin_3), J5.3 (Pin_3)
- net MCU_COL_2: now also J4.3 (Pin_3), J5.3 (Pin_3); no longer J4.4 (Pin_4), J5.4 (Pin_4)
- net MCU_COL_3: now also J4.6 (Pin_6), J5.6 (Pin_6); no longer J4.5 (Pin_5), J5.5 (Pin_5)
- net MCU_COL_4: now also J4.4 (Pin_4), J5.4 (Pin_4); no longer J4.6 (Pin_6), J5.6 (Pin_6)
- net at C12.1, R22.2: now also Q6.5 (D), Q6.6 (D), Q6.7 (D), Q6.8 (D); no longer Q6.1 (D)
- net at R3.2: now also Q6.4 (G); no longer Q6.3 (G)
- no-connect marks 36 -> 24
