File: kicad/hcms_dot_display/hcms_dot_display.kicad_sch (KiCad schematic)
At the start: 52 parts, among them J1 Conn_01x12, J2 USB_C_Receptacle_USB2.0, J3 Conn_01x12, J4 Conn_01x11_Female, J5 Conn_01x11_Male, J6 Conn_01x12, J7 Conn_01x12, Q1 Q_PMOS_DSG, Q2 Q_PMOS_DSG, Q3 Q_PMOS_DSG, Q4 Q_PMOS_DSG, Q5 Q_PMOS_DSG, Q6 Q_PMOS_DSG, SW1 SW_DIP_x03, U1 ATtiny826-SXX, U2 FT231XS

Commit message: layout ready for review i think
Parts:
- added J8: Conn_01x02_Male, Connector_PinHeader_2.54mm:PinHeader_1x02_P2.54mm_Vertical, symbol Connector:Conn_01x02_Male
- added MH1, MH2: MountingHole, MountingHole:MountingHole_2.2mm_M2_Pad_Via, symbol Mechanical:MountingHole
- added R23: 0, Resistor_SMD:R_0603_1608Metric, symbol Device:R
- U1: value ATtiny826-SXX -> ATtiny1626-X; footprint Package_SO:SOIC-20W_7.5x12.8mm_P1.27mm -> Package_SO:SSOP-20_5.3x7.2mm_P0.65mm
Connections:
- net +5V: now also R23.1
- net CONFIG_1: now also U1.4 (PA6); no longer U1.2 (PA4)
- net CONFIG_2: now also U1.2 (PA4); no longer U1.4 (PA6)
- net GND: now also J8.2 (Pin_2)
- new net: J8.1 (Pin_1), R23.2
Other:
- note added: "Backup power connection"
Changed lines of the file:
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@@
     (stroke (width 0) (type default) (color 0 0 0 0))
   )
+  (wire (pts (xy 28.575 172.72) (xy 28.575 175.895))
+    (stroke (width 0) (type default) (color 0 0 0 0))
+  )
   (wire (pts (xy 380.365 114.3) (xy 376.555 114.3))
     (stroke (width 0) (type default) (color 0 0 0 0))
@@
     (stroke (width 0) (type default) (color 0 0 0 0))
   )
+  (wire (pts (xy 36.195 170.18) (xy 39.37 170.18))
+    (stroke (width 0) (type default) (color 0 0 0 0))
+  )
   (wire (pts (xy 261.62 240.665) (xy 256.54 240.665))
     (stroke (width 0) (type default) (color 0 0 0 0))
@@
     (stroke (width 0) (type default) (color 0 0 0 0))
   )
+  (wire (pts (xy 39.37 167.005) (xy 39.37 170.18))
+    (stroke (width 0) (type default) (color 0 0 0 0))
+  )
   (wire (pts (xy 207.01 124.46) (xy 220.98 124.46))
     (stroke (width 0) (type default) (color 0 0 0 0))
@@
     (effects (font (size 1.27 1.27)) (justify left bottom))
   )
+  (text "Backup power connection" (at 22.86 154.305 0)
+    (effects (font (size 1.27 1.27)) (justify left bottom))
+  )
   (text "MIC5018YM4-TR" (at 156.845 126.365 0)
     (effects (font (size 1.27 1.27)) (justify left bottom))
@@
     (effects (font (size 4 4)) (justify left bottom))
   )
-  (label "CONFIG_2" (at 330.2 214.63 180)
+  (label "CONFIG_1" (at 330.2 214.63 180)
     (effects (font (size 1.27 1.27)) (justify right bottom))
   )
@@
     (effects (font (size 1.27 1.27)) (justify left bottom))
   )
-  (label "CONFIG_1" (at 330.2 209.55 180)
+  (label "CONFIG_2" (at 330.2 209.55 180)
     (effects (font (size 1.27 1.27)) (justify right bottom))
   )
@@
     (pin "2")
   )
+  (symbol (lib_id "Device:R") (at 32.385 170.18 270) (unit 1)
+    (in_bom yes) (on_board yes)
+    (property "Reference" "R23" (id 0) (at 29.845 168.91 90)
+      (effects (font (size 1.27 1.27)) (justify left bottom))
+    )
+    (property "Value" "0" (id 1) (at 29.845 171.45 90)
+      (effects (font (size 1.27 1.27)) (justify left top))
+    )
+    (property "Footprint" "Resistor_SMD:R_0603_1608Metric" (id 2) (at 32.385 168.402 90)
+      (effects (font (size 1.27 1.27)) hide)
+    )
+    (property "Datasheet" "~" (id 3) (at 32.385 170.18 0)
+      (effects (font (size 1.27 1.27)) hide)
+    )
+    (pin "1")
+    (pin "2")
+  )
   (symbol (lib_id "Device:R") (at 313.69 173.355 270) (unit 1)
     (in_bom yes) (on_board yes)
@@
     (pin "1")
   )
+  (symbol (lib_id "power:+5V") (at 39.37 167.005 0) (unit 1)
+    (in_bom yes) (on_board yes)
+    (property "Reference" "#PWR0129" (id 0) (at 39.37 170.815 0)
+      (effects (font (size 1.27 1.27)) hide)
+    )
+    (property "Value" "+5V" (id 1) (at 39.37 163.195 0))
+    (property "Footprint" "" (id 2) (at 39.37 167.005 0)
+      (effects (font (size 1.27 1.27)) hide)
+    )
+    (property "Datasheet" "" (id 3) (at 39.37 167.005 0)
+      (effects (font (size 1.27 1.27)) hide)
+    )
+    (pin "1")
+  )
   (symbol (lib_id "power:GND") (at 97.79 215.265 0) (unit 1)
     (in_bom yes) (on_board yes) (fields_autoplaced)
@@
     (pin "2")
   )
+  (symbol (lib_id "Connector:Conn_01x02_Male") (at 23.495 170.18 0) (unit 1)
+    (in_bom yes) (on_board yes)
+    (property "Reference" "J8" (id 0) (at 24.13 156.21 0))
+    (property "Value" "Conn_01x02_Male" (id 1) (at 22.86 158.75 0)
+      (effects (font (size 1.27 1.27)) (justify left))
+    )
+    (property "Footprint" "Connector_PinHeader_2.54mm:PinHeader_1x02_P2.54mm_Vertical" (id 2) (at 23.495 170.18 0)
+      (effects (font (size 1.27 1.27)) hide)
+    )
+    (property "Datasheet" "~" (id 3) (at 23.495 170.18 0)
+      (effects (font (size 1.27 1.27)) hide)
+    )
+    (pin "1")
+    (pin "2")
+  )
   (symbol (lib_id "Device:C_Small") (at 241.3 158.75 0) (unit 1)
     (in_bom yes) (on_board yes) (fields_autoplaced)
@@
     (pin "2")
   )
+  (symbol (lib_id "power:GND") (at 28.575 175.895 0) (unit 1)
+    (in_bom yes) (on_board yes) (fields_autoplaced)
+    (property "Reference" "#PWR0130" (id 0) (at 28.575 182.245 0)
+      (effects (font (size 1.27 1.27)) hide)
+    )
+    (property "Value" "GND" (id 1) (at 28.575 180.975 0))
+    (property "Footprint" "" (id 2) (at 28.575 175.895 0)
+      (effects (font (size 1.27 1.27)) hide)
+    )
+    (property "Datasheet" "" (id 3) (at 28.575 175.895 0)
+      (effects (font (size 1.27 1.27)) hide)
+    )
+    (pin "1")
+  )
   (symbol (lib_id "power:GND") (at 277.495 236.22 0) (unit 1)
     (in_bom yes) (on_board yes)
@@
     (pin "8A")
     (pin "9A")
-    (pin "10B")
-    (pin "12B")
-    (pin "13B")
-    (pin "14B")
-    (pin "15B")
-    (pin "17B")
-    (pin "18B")
-    (pin "19B")
-    (pin "1B")
-    (pin "21B")
-    (pin "22B")
-    (pin "23B")
-    (pin "25B")
-    (pin "26B")
-    (pin "2B")
-    (pin "4B")
-    (pin "5B")
-    (pin "6B")
-    (pin "8B")
-    (pin "9B")
   )
   (symbol (lib_id "power:GND") (at 165.735 260.35 0) (unit 1)
@@
     (pin "1")
   )
+  (symbol (lib_id "Mechanical:MountingHole") (at 92.075 161.29 0) (unit 1)
+    (in_bom yes) (on_board yes) (fields_autoplaced)
+    (property "Reference" "MH2" (id 0) (at 95.25 160.0199 0)
+      (effects (font (size 1.27 1.27)) (justify left))
+    )
+    (property "Value" "MountingHole" (id 1) (at 95.25 162.5599 0)
+      (effects (font (size 1.27 1.27)) (justify left))
+    )
+    (property "Footprint" "MountingHole:MountingHole_2.2mm_M2_Pad_Via" (id 2) (at 92.075 161.29 0)
+      (effects (font (size 1.27 1.27)) hide)
+    )
+    (property "Datasheet" "~" (id 3) (at 92.075 161.29 0)
+      (effects (font (size 1.27 1.27)) hide)
+    )
+  )
   (symbol (lib_id "power:GND") (at 136.525 210.185 0) (unit 1)
     (in_bom yes) (on_board yes) (fields_autoplaced)
@@
     (pin "1")
   )
+  (symbol (lib_id "Mechanical:MountingHole") (at 71.12 161.29 0) (unit 1)
+    (in_bom yes) (on_board yes) (fields_autoplaced)
+    (property "Reference" "MH1" (id 0) (at 73.66 160.0199 0)
+      (effects (font (size 1.27 1.27)) (justify left))
+    )
+    (property "Value" "MountingHole" (id 1) (at 73.66 162.5599 0)
+      (effects (font (size 1.27 1.27)) (justify left))
+    )
+    (property "Footprint" "MountingHole:MountingHole_2.2mm_M2_Pad_Via" (id 2) (at 71.12 161.29 0)
+      (effects (font (size 1.27 1.27)) hide)
+    )
+    (property "Datasheet" "~" (id 3) (at 71.12 161.29 0)
+      (effects (font (size 1.27 1.27)) hide)
+    )
+  )
   (symbol (lib_id "Device:R") (at 224.155 69.85 270) (unit 1)
     (in_bom yes) (on_board yes)
@@
       (effects (font (size 1.27 1.27)) hide)
     )
-    (pin "10A")
-    (pin "12A")
-    (pin "13A")
-    (pin "14A")
-    (pin "15A")
-    (pin "17A")
-    (pin "18A")
-    (pin "19A")
-    (pin "1A")
-    (pin "21A")
-    (pin "22A")
-    (pin "23A")
-    (pin "25A")
-    (pin "26A")
-    (pin "2A")
-    (pin "4A")
-    (pin "5A")
-    (pin "6A")
-    (pin "8A")
-    (pin "9A")
     (pin "10B")
     (pin "12B")
@@
     (in_bom yes) (on_board yes) (fields_autoplaced)
     (property "Reference" "U1" (id 0) (at 297.18 190.5 0))
-    (property "Value" "ATtiny826-SXX" (id 1) (at 297.18 193.04 0))
-    (property "Footprint" "Package_SO:SOIC-20W_7.5x12.8mm_P1.27mm" (id 2) (at 304.8 243.84 0)
+    (property "Value" "ATtiny1626-X" (id 1) (at 297.18 193.04 0))
+    (property "Footprint" "Package_SO:SSOP-20_5.3x7.2mm_P0.65mm" (id 2) (at 304.8 243.84 0)
       (effects (font (size 1.27 1.27) italic) hide)
     )
@@
       (reference "#PWR0128") (unit 1) (value "GND") (footprint "")
     )
+    (path "/1b2fbf52-6faa-4937-83fa-9387d825d297"
+      (reference "#PWR0129") (unit 1) (value "+5V") (footprint "")
+    )
+    (path "/7e4d40de-ad0c-4cd2-bc51-b5dd40e98c5e"
+      (reference "#PWR0130") (unit 1) (value "GND") (footprint "")
+    )
     (path "/a585cb01-913c-4013-af5c-5954c151d6ce"
       (reference "C1") (unit 1) (value "10nF") (footprint "Capacitor_SMD:C_0603_1608Metric")
@@
       (reference "J7") (unit 1) (value "Conn_01x12") (footprint "hcms:board to board con left right")
     )
+    (path "/7b38995c-2cf1-4790-9813-32dbe6381c9d"
+      (reference "J8") (unit 1) (value "Conn_01x02_Male") (footprint "Connector_PinHeader_2.54mm:PinHeader_1x02_P2.54mm_Vertical")
+    )
+    (path "/b94ee3bb-9400-43cc-a324-ca6d75f88eed"
+      (reference "MH1") (unit 1) (value "MountingHole") (footprint "MountingHole:MountingHole_2.2mm_M2_Pad_Via")
+    )
+    (path "/9ff1ec12-e027-4234-aae5-627f439427d4"
+      (reference "MH2") (unit 1) (value "MountingHole") (footprint "MountingHole:MountingHole_2.2mm_M2_Pad_Via")
+    )
     (path "/cb19c6f6-ba2e-40c5-b24e-87d5c3df300e"
       (reference "Q1") (unit 1) (value "Q_PMOS_DSG") (footprint "Package_TO_SOT_SMD:SOT-23")
@@
       (reference "R22") (unit 1) (value "0") (footprint "Resistor_SMD:R_0603_1608Metric")
     )
+    (path "/067a4263-aa80-426a-8cd2-15ee22505f70"
+      (reference "R23") (unit 1) (value "0") (footprint "Resistor_SMD:R_0603_1608Metric")
+    )
     (path "/26df86c2-e6da-4304-8085-b1a7b60b8ac0"
       (reference "RV1") (unit 1) (value "R_Potentiometer") (footprint "hcms:TRIM_3352T-1-201LF")
@@
     )
     (path "/ec702393-b640-4b47-ba2e-5eeb75d59724"
-      (reference "U1") (unit 1) (value "ATtiny826-SXX") (footprint "Package_SO:SOIC-20W_7.5x12.8mm_P1.27mm")
+      (reference "U1") (unit 1) (value "ATtiny1626-X") (footprint "Package_SO:SSOP-20_5.3x7.2mm_P0.65mm")
     )
     (path "/34ae76d3-991a-467a-bf8f-43f39fb1570d"
