File: kicad/hcms_dot_display_bottom/hcms_dot_display_bottom.kicad_sch (KiCad schematic)
At the start: 56 parts, among them J1 Conn_01x12, J2 USB_C_Receptacle_USB2.0, J3 Conn_01x12, J4 Conn_01x11_Female, J5 Conn_01x11_Male, J6 Conn_01x12, J7 Conn_01x12, J8 Conn_01x02_Male, Q1 Q_PMOS_DSG, Q2 Q_PMOS_DSG, Q3 Q_PMOS_DSG, Q4 Q_PMOS_DSG, Q5 Q_PMOS_DSG, Q6 Q_PMOS_DSG, SW1 SW_DIP_x03, U1 ATtiny1626-X, U2 FT231XS

Commit message: progress making bottom manufacturable
Parts:
- removed C10, C11: 10nF, Capacitor_SMD:C_0603_1608Metric, symbol Device:C_Small
- removed C3: 100nF, Capacitor_SMD:C_0603_1608Metric, symbol Device:C_Small
- removed D1: HCMS-272X, hcms:HCMS-2722, symbol hcms_dot_display:HCMS-272X
- removed J1, J3: Conn_01x12, hcms:board to board con top bot, symbol Connector_Generic:Conn_01x12
- removed J5: Conn_01x11_Male, Connector_PinHeader_2.54mm:PinHeader_1x11_P2.54mm_Vertical, symbol Connector:Conn_01x11_Male
- removed J6, J7: Conn_01x12, hcms:board to board con left right, symbol Connector_Generic:Conn_01x12
- removed Q1, Q2, Q3, Q4, Q5: Q_PMOS_DSG, Package_TO_SOT_SMD:SOT-23, symbol Device:Q_PMOS_DSG
- removed R1, R6: 0, Resistor_SMD:R_0603_1608Metric, symbol Device:R
- removed R10, R11, R12, R13, R14: 200, Resistor_SMD:R_0603_1608Metric, symbol Device:R
- removed R16, R17, R2, R7: DNP, Resistor_SMD:R_0603_1608Metric, symbol Device:R
- renumbered J4 to J5
Connections:
- no-connect marks 24 -> 16
Other:
- note removed: "BOARD 1 A_DATA -> BOARD 2 DAISY_A_DATA"
- note removed: "BOARD 1 B_DATA -> BOARD 2 DAISY_B_DATA"
- note removed: "DMN2046U"
- note removed: "INCOMING SIGNALS"
- note removed: "MIC5018YM4-TR"
- note removed: "OUTGOING SIGNALS"
- note removed: "TOP PCB"
- moved on the sheet: C1, C12, C2, C4, C5, C6, C7, C8, C9, J2, J5, J8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
