File: kicad/hcms_dot_display_top/_autosave-hcms_dot_display_top.kicad_sch (KiCad schematic)
At the start: 25 parts, among them J1 Conn_01x12, J3 Conn_01x12, J4 Conn_01x11_Male, J6 Conn_01x12, J7 Conn_01x12, Q1 Q_PMOS_GSD, Q2 Q_PMOS_GSD, Q3 Q_PMOS_GSD, Q4 Q_PMOS_GSD, Q5 Q_PMOS_GSD

Commit message: Fixed daisy issue left right
Connections:
- net A_DATA: now also J7.10 (Pin_10); no longer J6.10 (Pin_10)
- net B_DATA: now also J7.11 (Pin_11); no longer J6.11 (Pin_11)
- net DAISY_A_DATA: now also J6.10 (Pin_10); no longer J7.10 (Pin_10)
- net DAISY_B_DATA: now also J6.11 (Pin_11); no longer J7.11 (Pin_11)
Changed lines of the file:
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@@
     (effects (font (size 1.27 1.27)) (justify left bottom))
   )
-  (label "A_DATA" (at 24.13 174.625 0)
-    (effects (font (size 1.27 1.27)) (justify left bottom))
+  (label "A_DATA" (at 396.24 173.355 180)
+    (effects (font (size 1.27 1.27)) (justify right bottom))
   )
   (label "MCU_COL_3" (at 396.24 116.205 180)
@@
     (effects (font (size 1.27 1.27)) (justify left bottom))
   )
-  (label "DAISY_B_DATA" (at 396.24 175.895 180)
-    (effects (font (size 1.27 1.27)) (justify right bottom))
+  (label "DAISY_B_DATA" (at 24.13 177.165 0)
+    (effects (font (size 1.27 1.27)) (justify left bottom))
   )
   (label "CLK" (at 24.13 172.085 0)
@@
     (effects (font (size 1.27 1.27)) (justify left bottom))
   )
-  (label "B_DATA" (at 24.13 177.165 0)
-    (effects (font (size 1.27 1.27)) (justify left bottom))
+  (label "B_DATA" (at 396.24 175.895 180)
+    (effects (font (size 1.27 1.27)) (justify right bottom))
   )
   (label "COL_2" (at 241.3 160.02 0)
@@
     (effects (font (size 1.27 1.27)) (justify left bottom))
   )
-  (label "DAISY_A_DATA" (at 396.24 173.355 180)
-    (effects (font (size 1.27 1.27)) (justify right bottom))
+  (label "DAISY_A_DATA" (at 24.13 174.625 0)
+    (effects (font (size 1.27 1.27)) (justify left bottom))
   )
   (label "COL_5" (at 241.3 167.64 0)
